Commit message: Add the lieDown spawn posture, damp the trunk contact
- lieDown group state: on the belly, legs folded, feet just off the ground;
  the rl_quadruped controller spawns in it.
- go0 takes the group state from its go0_conf argument (default home), and
  takes the first joint readings in a staged posture: gazebo_ros_control
  starts every reading at 1 rad and unwraps from there, so a knee spawned
  below 1 - pi read 2 pi too high for the whole run.
- The trunk gets the feet's contact kp/kd: undamped, the lying body chattered
  on the ground and spoiled the IMU calibration.

File: robots/aliengo.srdf.xacro (robot description, xacro)
@@ -63,4 +63,19 @@
         <joint name="rh_kfe_joint" value="-1.4"/>
     </group_state>
+    <!-- on the belly, legs folded, feet just off the ground (rl_quadruped spawn) -->
+    <group_state group="chains" name="lieDown">
+        <joint name="lf_haa_joint" value="0.65"/>
+        <joint name="lf_hfe_joint" value="1.38"/>
+        <joint name="lf_kfe_joint" value="-2.75"/>
+        <joint name="rf_haa_joint" value="-0.65"/>
+        <joint name="rf_hfe_joint" value="1.38"/>
+        <joint name="rf_kfe_joint" value="-2.75"/>
+        <joint name="lh_haa_joint" value="0.65"/>
+        <joint name="lh_hfe_joint" value="1.38"/>
+        <joint name="lh_kfe_joint" value="-2.75"/>
+        <joint name="rh_haa_joint" value="-0.65"/>
+        <joint name="rh_hfe_joint" value="1.38"/>
+        <joint name="rh_kfe_joint" value="-2.75"/>
+    </group_state>
     <group_state group="chains" name="home">
         <joint name="lf_haa_joint" value="0.80"/>

File: robots/aliengo.urdf.xacro (robot description, xacro)
@@ -188,3 +188,9 @@
 	    </gazebo>
     </xacro:if>
+    <!-- Body contacts damped like the feet: undamped, the body chatters on the ground while the
+         robot lies and the accelerometer calibration never settles. -->
+    <gazebo reference="trunk">
+        <kp>1000000.0</kp>
+        <kd>${contact_kd}</kd>
+    </gazebo>
 </robot>

File: urdfs/const.xacro (robot description, xacro)
@@ -40,5 +40,5 @@
     <xacro:property name="joint_viscous" value="${dict(haa=0.29, hfe=0.26, kfe=0.3)}"/>
     <xacro:property name="joint_armature" value="${dict(haa=0.0023, hfe=0.014, kfe=0.015)}"/>
-    <!-- Contact damping, N s/m (leg.gazebo.xacro): at 100 the feet bounce on touchdown. -->
+    <!-- Contact damping, N s/m (leg.gazebo.xacro and the body): at 100 the feet bounce on touchdown. -->
     <xacro:property name="contact_kd" value="3000.0"/>
     <xacro:property name="HAA_position_max" value="${70*PI/180.0}"/>
